File: DigitalClock.kicad_sch (KiCad schematic)
At the start: 11 parts

Commit message: Updated Schematic
Other:
- company: (none) -> Sunnickel
- title: (none) -> Digital Clock
Changed lines of the file:
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@@
 	(generator_version "9.0")
 	(paper "A4")
+	(title_block
+		(title "Digital Clock")
+		(date "2025-07-06")
+		(company "Sunnickel")
+	)
 	(junction
 		(at 45.72 114.3)
